Commit message: Created Gazebo world, modified URDFs accordingly

File: description/robot_core.xacro (robot description, xacro)
@@ -43,4 +43,9 @@
         </xacro:inertial_box>
     </link>
+    <gazebo reference="chassis">
+        <material>
+            Gazebo/White
+        </material>
+    </gazebo>
     <!-- Left Wheel Link > lengths are in meters! -->
     <joint name="left_wheel_joint" type="continuous">
@@ -68,4 +73,9 @@
         </xacro:inertial_cylinder>
     </link>
+    <gazebo reference="left_wheel">
+        <material>
+            Gazebo/Blue
+        </material>
+    </gazebo>
     <!-- Right Wheel Link > lengths are in meters! -->
     <joint name="right_wheel_joint" type="continuous">
@@ -94,4 +104,9 @@
         </xacro:inertial_cylinder>
     </link>
+    <gazebo reference="right_wheel">
+        <material>
+            Gazebo/Blue
+        </material>
+    </gazebo>
     <!-- Caster Wheel Link -->
     <joint name="caster_wheel_joint" type="fixed">
@@ -117,3 +132,11 @@
         </xacro:inertial_sphere>
     </link>
+    <gazebo reference="caster_wheel">
+        <material>
+            Gazebo/Black
+        </material>
+        <!-- adding friction coefficient(katsayı). not mul, mu1 (one)!-->
+        <mu1 value = "0.001"/>
+        <mu2 value = "0.001"/>
+    </gazebo>
 </robot>

Commit message: Added some comments, changed colors

File: description/robot_core.xacro (robot description, xacro)
@@ -30,5 +30,5 @@
                 <box size="0.3 0.3 0.15"/>
             </geometry>
-            <material name="white"/>
+            <material name="orange"/>
         </visual>
         <collision>
@@ -45,5 +45,5 @@
     <gazebo reference="chassis">
         <material>
-            Gazebo/White
+            Gazebo/Orange
         </material>
     </gazebo>

Commit message: Added lidar

File: description/robot_core.xacro (robot description, xacro)
@@ -13,4 +13,7 @@
     <material name="orange">
         <color rgba="1.0 0.3 0.1 1.0"/>
+    </material>
+    <material name="red">
+        <color rgba="1.0 0.0 0.0 1.0"/>
     </material>
     <!-- Base Link -->

Commit message: Added base_footprint to robot_core

File: description/robot_core.xacro (robot description, xacro)
@@ -19,4 +19,13 @@
     <!-- Base Link -->
     <link name="base_link">
+    </link>
+    <!-- Base Footprint for SLAM -->
+    <!-- base footprint must be treated like it's on the floor. Our example robot is basically on the floor so we can treat it so -->
+    <joint name="base_footprint_joint" type="fixed">
+        <parent link="base_link"/>
+        <child link="base_footprint"/>
+        <origin xyz="0 0 0" rpy="0 0 0"/>
+    </joint>
+    <link name="base_footprint">
     </link>
     <!-- Chassis Joint / Link -->
